Commit message: minimal working structure

File: workspace/upper_body_teleop_home_full/src/humanoid_description_ros2/urdf/full_humanoid_upper_body.urdf (robot description, URDF)
Before this commit: robot full_humanoid_upper_body_test, 25 links, 24 joints
Joints:
- joint left_shoulder_pitch_joint: axis 0 1 0 -> 0 0 1
- joint left_shoulder_yaw_joint: axis 0 0 1 -> 0 1 0
- joint right_shoulder_pitch_joint: axis 0 1 0 -> 0 0 1
- joint right_shoulder_yaw_joint: axis 0 0 1 -> 0 -1 0
